Commit message: gripper added, joint state brodcaster, trajectory controller added

File: my_robotic_arm/urdf/Arm_Urdf.urdf (robot description, URDF)
Before this commit: robot Arm_Urdf, 18 links, 17 joints
Links:
- removed link pointer_base
- removed link pointer_tip
- added link Gripper_1, mass 0.137742996071251; collision mesh filename=package://my_robotic_arm/meshes/Gripper_1.STL; visual mesh filename=package://my_robotic_arm/meshes/Gripper_1.STL
- added link Gripper_2, mass 0.153524806277575; collision mesh filename=package://my_robotic_arm/meshes/Gripper_2.STL; visual mesh filename=package://my_robotic_arm/meshes/Gripper_2.STL
Joints:
- removed joint pointer_base_joint
- removed joint pointer_extend_joint
- added joint Finger_1: type prismatic, parent Link_6, child Gripper_1, origin xyz=0.00534999999999963 -0.0390954035350414 0.0487946645392847 rpy=1.5707963267949 0 1.5707963267949, axis 0 0 -1, limit lower=0 upper=0.0355 effort=100 velocity=10
- added joint Finger_2: type prismatic, parent Link_6, child Gripper_2, origin xyz=0.00534999999999963 -0.0390954035350414 0.0487946645392847 rpy=1.5707963267949 0 1.5707963267949, axis 0 0 -1, limit lower=-0.0355 upper=0 effort=100 velocity=10
